File: Schemas/CardReader/cardReader.sch (KiCad schematic (older format))
At the start: 29 parts, among them P1 PWR, P2 DATA, Q1 BC817-40, U1 74HC165

Commit message: Update cardReader schema, add end pin
Parts:
- P2: footprint Pin_Headers:Pin_Header_Straight_1x04_Pitch2.54mm -> Pin_Headers:Pin_Header_Straight_1x05_Pitch2.54mm; symbol CONN_01X04 -> CONN_01X05
Connections:
- net gnd: now also P2.5 (P5)
Changed lines of the file:
@@
 Connection ~ 1700 1250
 $Comp
-L CONN_01X04 P2
+L CONN_01X05 P2
 U 1 1 589B659E
-P 4550 5100
-F 0 "P2" H 4550 5350 50  0000 C CNN
-F 1 "DATA" V 4650 5100 50  0000 C CNN
-F 2 "Pin_Headers:Pin_Header_Straight_1x04_Pitch2.54mm" H 4550 5100 50  0001 C CNN
-F 3 "" H 4550 5100 50  0000 C CNN
-	1    4550 5100
+P 4500 5100
+F 0 "P2" H 4500 5350 50  0000 C CNN
+F 1 "DATA" V 4600 5100 50  0000 C CNN
+F 2 "Pin_Headers:Pin_Header_Straight_1x05_Pitch2.54mm" H 4500 5100 50  0001 C CNN
+F 3 "" H 4500 5100 50  0000 C CNN
+	1    4500 5100
 	0    1    1    0
 $EndComp
@@
 Wire Wire Line
 	1550 1450 1950 1450
+Wire Wire Line
+	4300 4900 4300 4550
+Wire Wire Line
+	4300 4550 1600 4550
+Wire Wire Line
+	1600 4550 1600 1450
+Connection ~ 1600 1450
 $EndSCHEMATC
